Commit message: Add an "is_sim" flag to the Kobuki urdf.
This flag is used to determine whether to use the Gazebo plugin for simulating data.

File: kobuki_ws/src/kobuki_ros/kobuki_description/urdf/kobuki.urdf.xacro (robot description, xacro)
@@ -10,5 +10,5 @@
   <xacro:include filename="$(find kobuki_description)/urdf/kobuki_gazebo.urdf.xacro"/>
   <!-- Kobuki -->
-  <xacro:macro name="kobuki">
+  <xacro:macro name="kobuki" params="is_sim:=true">
     <link name="base_footprint"/>
     <!--
@@ -209,5 +209,7 @@
     </link>
     <!-- Kobuki Gazebo simulation details -->
-    <xacro:kobuki_sim/>
+    <xacro:if value="$(arg is_sim)">
+        <xacro:kobuki_sim/>
+    </xacro:if>
   </xacro:macro>
 </robot>

File: kobuki_ws/src/kobuki_ros/kobuki_description/urdf/kobuki_VLP16.urdf.xacro (robot description, xacro)
@@ -1,15 +1,23 @@
 <?xml version="1.0"?>
 <robot name="kobuki_VLP16" xmlns:xacro="http://ros.org/wiki/xacro">
+    <!-- Arguments -->
+    <xacro:arg name="is_sim" default="true"/>
+    <xacro:arg name="VLP16_enabled" default="true"/>
     <xacro:arg name="gpu" default="false"/>
     <xacro:arg name="organize_cloud" default="false"/>
-    <xacro:property name="gpu" value="$(arg gpu)" />
-    <xacro:property name="organize_cloud" value="$(arg organize_cloud)" />
+    <!-- Properties -->
+    <xacro:property name="is_sim" value="$(arg is_sim)"/>
+    <xacro:property name="VLP16_enabled" value="$(arg VLP16_enabled)"/>
+    <xacro:property name="gpu" value="$(arg gpu)"/>
+    <xacro:property name="organize_cloud" value="$(arg organize_cloud)"/>
     <!-- Defines the kobuki component tag. -->
     <xacro:include filename="$(find kobuki_description)/urdf/kobuki.urdf.xacro" />
-    <xacro:kobuki/>
+    <xacro:kobuki is_sim="${is_sim}"/>
     <!-- Defines the VLP-16 component tag. -->
-    <xacro:include filename="$(find velodyne_description)/urdf/VLP-16.urdf.xacro"/>
-    <xacro:VLP-16 parent="base_link" name="velodyne" topic="/velodyne_points" organize_cloud="${organize_cloud}" hz="10" samples="440" gpu="${gpu}">
-        <origin xyz="0 0 0.4" rpy="0 0 0" />
-    </xacro:VLP-16>
+    <xacro:if value="$(arg VLP16_enabled)">
+        <xacro:include filename="$(find velodyne_description)/urdf/VLP-16.urdf.xacro"/>
+        <xacro:VLP-16 is_sim="${is_sim}" parent="base_link" name="velodyne" topic="/velodyne_points" organize_cloud="${organize_cloud}" hz="10" samples="440" gpu="${gpu}">
+            <origin xyz="0 0 0.4" rpy="0 0 0" />
+        </xacro:VLP-16>
+    </xacro:if>
 </robot>

File: kobuki_ws/src/kobuki_ros/kobuki_description/urdf/kobuki_standalone.urdf.xacro (robot description, xacro)
@@ -1,10 +1,10 @@
 <?xml version="1.0"?>
-<robot name="kobuki_standalone"
-       xmlns:sensor="http://playerstage.sourceforge.net/gazebo/xmlschema/#sensor"
-       xmlns:controller="http://playerstage.sourceforge.net/gazebo/xmlschema/#controller"
-       xmlns:interface="http://playerstage.sourceforge.net/gazebo/xmlschema/#interface"
-       xmlns:xacro="http://ros.org/wiki/xacro">
-  <!-- Defines the kobuki component tag. -->
-  <xacro:include filename="$(find kobuki_description)/urdf/kobuki.urdf.xacro" />
-  <xacro:kobuki/>
+<robot name="kobuki_standalone">
+    <!-- Arguments -->
+    <xacro:arg name="is_sim" default="true"/>
+    <!-- Properties -->
+    <xacro:property name="is_sim" value="$(arg is_sim)" />
+    <!-- Defines the kobuki component tag. -->
+    <xacro:include filename="$(find kobuki_description)/urdf/kobuki.urdf.xacro" />
+    <xacro:kobuki is_sim="${is_sim}"/>
 </robot>

File: kobuki_ws/src/velodyne_simulator/velodyne_description/urdf/VLP-16.urdf.xacro (robot description, xacro)
@@ -2,5 +2,5 @@
 <robot xmlns:xacro="http://www.ros.org/wiki/xacro" name="VLP-16">
   <xacro:property name="M_PI" value="3.1415926535897931" />
-  <xacro:macro name="VLP-16" params="*origin parent:=base_link name:=velodyne tf_prefix:='' topic:=/velodyne_points organize_cloud:=false hz:=10 lasers:=16 samples:=1875 collision_range:=0.3 min_range:=0.9 max_range:=130.0 noise:=0.008 min_angle:=-${M_PI} max_angle:=${M_PI} gpu:=false">
+  <xacro:macro name="VLP-16" params="*origin is_sim:=true parent:=base_link name:=velodyne tf_prefix:='' topic:=/velodyne_points organize_cloud:=false hz:=10 lasers:=16 samples:=1875 collision_range:=0.3 min_range:=0.9 max_range:=130.0 noise:=0.008 min_angle:=-${M_PI} max_angle:=${M_PI} gpu:=false">
     <joint name="${name}_base_mount_joint" type="fixed">
       <xacro:insert_block name="origin" />
@@ -57,96 +57,98 @@
     </link>
     <!-- Gazebo requires the velodyne_gazebo_plugins package -->
-    <gazebo reference="${name}">
-      <xacro:if value="${gpu}">
-        <sensor type="gpu_ray" name="${name}-VLP16">
-          <pose>0 0 0 0 0 0</pose>
-          <visualize>false</visualize>
-          <update_rate>${hz}</update_rate>
-          <ray>
-            <scan>
-              <horizontal>
-                <samples>${samples}</samples>
-                <resolution>1</resolution>
-                <min_angle>${min_angle}</min_angle>
-                <max_angle>${max_angle}</max_angle>
-              </horizontal>
-              <vertical>
-                <samples>${lasers}</samples>
-                <resolution>1</resolution>
-                <min_angle>-${15.0*M_PI/180.0}</min_angle>
-                <max_angle> ${15.0*M_PI/180.0}</max_angle>
-              </vertical>
-            </scan>
-            <range>
-              <min>${collision_range}</min>
-              <max>${max_range+1}</max>
-              <resolution>0.001</resolution>
-            </range>
-            <noise>
-              <type>gaussian</type>
-              <mean>0.0</mean>
-              <stddev>0.0</stddev>
-            </noise>
-          </ray>
-          <plugin name="gazebo_ros_laser_controller" filename="libgazebo_ros_velodyne_laser.so">
-            <ros>
-              <namespace>/${name}</namespace>
-              <remapping>~/out:=${topic}</remapping>
-            </ros>
-            <tf_prefix>${tf_prefix}</tf_prefix>
-            <frame_name>${name}</frame_name>
-            <organize_cloud>${organize_cloud}</organize_cloud>
-            <min_range>${min_range}</min_range>
-            <max_range>${max_range}</max_range>
-            <gaussian_noise>${noise}</gaussian_noise>
-          </plugin>
-        </sensor>
-      </xacro:if>
-      <xacro:unless value="${gpu}">
-        <sensor type="ray" name="${name}-VLP16">
-          <pose>0 0 0 0 0 0</pose>
-          <visualize>false</visualize>
-          <update_rate>${hz}</update_rate>
-          <ray>
-            <scan>
-              <horizontal>
-                <samples>${samples}</samples>
-                <resolution>1</resolution>
-                <min_angle>${min_angle}</min_angle>
-                <max_angle>${max_angle}</max_angle>
-              </horizontal>
-              <vertical>
-                <samples>${lasers}</samples>
-                <resolution>1</resolution>
-                <min_angle>-${15.0*M_PI/180.0}</min_angle>
-                <max_angle> ${15.0*M_PI/180.0}</max_angle>
-              </vertical>
-            </scan>
-            <range>
-              <min>${collision_range}</min>
-              <max>${max_range+1}</max>
-              <resolution>0.001</resolution>
-            </range>
-            <noise>
-              <type>gaussian</type>
-              <mean>0.0</mean>
-              <stddev>0.0</stddev>
-            </noise>
-          </ray>
-          <plugin name="gazebo_ros_laser_controller" filename="libgazebo_ros_velodyne_laser.so">
-            <ros>
-              <namespace>/${name}</namespace>
-              <remapping>~/out:=${topic}</remapping>
-            </ros>
-            <tf_prefix>${tf_prefix}</tf_prefix>
-            <frame_name>${name}</frame_name>
-            <organize_cloud>${organize_cloud}</organize_cloud>
-            <min_range>${min_range}</min_range>
-            <max_range>${max_range}</max_range>
-            <gaussian_noise>${noise}</gaussian_noise>
-          </plugin>
-        </sensor>
-      </xacro:unless>
-    </gazebo>
+    <xacro:if value="${is_sim}">
+        <gazebo reference="${name}">
+            <xacro:if value="${gpu}">
+                <sensor type="gpu_ray" name="${name}-VLP16">
+                <pose>0 0 0 0 0 0</pose>
+                <visualize>false</visualize>
+                <update_rate>${hz}</update_rate>
+                <ray>
+                    <scan>
+                    <horizontal>
+                        <samples>${samples}</samples>
+                        <resolution>1</resolution>
+                        <min_angle>${min_angle}</min_angle>
+                        <max_angle>${max_angle}</max_angle>
+                    </horizontal>
+                    <vertical>
+                        <samples>${lasers}</samples>
+                        <resolution>1</resolution>
+                        <min_angle>-${15.0*M_PI/180.0}</min_angle>
+                        <max_angle> ${15.0*M_PI/180.0}</max_angle>
+                    </vertical>
+                    </scan>
+                    <range>
+                    <min>${collision_range}</min>
+                    <max>${max_range+1}</max>
+                    <resolution>0.001</resolution>
+                    </range>
+                    <noise>
+                    <type>gaussian</type>
+                    <mean>0.0</mean>
+                    <stddev>0.0</stddev>
+                    </noise>
+                </ray>
+                <plugin name="gazebo_ros_laser_controller" filename="libgazebo_ros_velodyne_laser.so">
+                    <ros>
+                    <namespace>/${name}</namespace>
+                    <remapping>~/out:=${topic}</remapping>
+                    </ros>
+                    <tf_prefix>${tf_prefix}</tf_prefix>
+                    <frame_name>${name}</frame_name>
+                    <organize_cloud>${organize_cloud}</organize_cloud>
+                    <min_range>${min_range}</min_range>
+                    <max_range>${max_range}</max_range>
+                    <gaussian_noise>${noise}</gaussian_noise>
+                </plugin>
+                </sensor>
+            </xacro:if>
+            <xacro:unless value="${gpu}">
+                <sensor type="ray" name="${name}-VLP16">
+                <pose>0 0 0 0 0 0</pose>
+                <visualize>false</visualize>
+                <update_rate>${hz}</update_rate>
+                <ray>
+                    <scan>
+                    <horizontal>
+                        <samples>${samples}</samples>
+                        <resolution>1</resolution>
+                        <min_angle>${min_angle}</min_angle>
+                        <max_angle>${max_angle}</max_angle>
+                    </horizontal>
+                    <vertical>
+                        <samples>${lasers}</samples>
+                        <resolution>1</resolution>
+                        <min_angle>-${15.0*M_PI/180.0}</min_angle>
+                        <max_angle> ${15.0*M_PI/180.0}</max_angle>
+                    </vertical>
+                    </scan>
+                    <range>
+                    <min>${collision_range}</min>
+                    <max>${max_range+1}</max>
+                    <resolution>0.001</resolution>
+                    </range>
+                    <noise>
+                    <type>gaussian</type>
+                    <mean>0.0</mean>
+                    <stddev>0.0</stddev>
+                    </noise>
+                </ray>
+                <plugin name="gazebo_ros_laser_controller" filename="libgazebo_ros_velodyne_laser.so">
+                    <ros>
+                    <namespace>/${name}</namespace>
+                    <remapping>~/out:=${topic}</remapping>
+                    </ros>
+                    <tf_prefix>${tf_prefix}</tf_prefix>
+                    <frame_name>${name}</frame_name>
+                    <organize_cloud>${organize_cloud}</organize_cloud>
+                    <min_range>${min_range}</min_range>
+                    <max_range>${max_range}</max_range>
+                    <gaussian_noise>${noise}</gaussian_noise>
+                </plugin>
+                </sensor>
+            </xacro:unless>
+        </gazebo>
+    </xacro:if>
   </xacro:macro>
 </robot>

Commit message: Correct the TF frame hierarchy.
As specified in REP-120, the `base_link` should be the root, with all other links as its children.

Reference: https://www.ros.org/reps/rep-0120.html#frame-hierarchy

File: kobuki_ws/src/kobuki_ros/kobuki_description/urdf/kobuki.urdf.xacro (robot description, xacro)
@@ -19,10 +19,10 @@
        To put the base link at the more oft used wheel
        axis, set the z-distance from the base_footprint
-       to 0.352.
+       to -0.352.
       -->
     <joint name="base_joint" type="fixed">
-      <origin xyz="0 0 0.0102" rpy="0 0 0" />
-      <parent link="base_footprint"/>
-      <child link="base_link" />
+      <origin xyz="0 0 -0.0102" rpy="0 0 0" />
+      <parent link="base_link" />
+      <child link="base_footprint" />
     </joint>
     <link name="base_link">

File: kobuki_ws/src/kobuki_ros/kobuki_description/urdf/kobuki_gazebo.urdf.xacro (robot description, xacro)
@@ -184,5 +184,5 @@
         <odometry_topic>odom</odometry_topic>
         <odometry_frame>odom</odometry_frame>
-        <robot_base_frame>base_footprint</robot_base_frame>
+        <robot_base_frame>base_link</robot_base_frame>
 	    </plugin>
 	  </gazebo>
